File: polivoks ambika.brd (EAGLE design)
At the start: 118.7 x 60.3 mm, 73 parts, among them IC1 TL084, IC10 LM4250P, IC11 LM13700N, IC2 4052N, IC5 TL072, IC6 MCP4822, IC7 ATMega328p, IC9 LM4250P, Q1 2N3906, Q2 2N3906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

Commit message: Added a resistor to limit the current on BP mode
Parts:
- added R3: 1k, rcl:0204/7
- moved Q4 5.39 mm to (59.7, 24.8)
Connections:
- new net N$23: IC7.23, R3.1
- net N$21: now also R3.2; no longer IC7.23
Routing:
- net SW: track 29.9 -> 34.1 mm
- net N$23: track 0.00 -> 3.81 mm
- net N$21: track 4.44 -> 6.02 mm
Changed lines of the file:
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@@
 </element>
 <element name="IC2" library="40xx" package="DIL16" value="4052N" x="66.04" y="40.64"/>
-<element name="Q4" library="transistor" package="TO92" value="2N3904" x="63.5" y="20.955" smashed="yes">
-<attribute name="NAME" x="57.785" y="20.955" size="1.27" layer="25" ratio="12"/>
-<attribute name="VALUE" x="54.61" y="19.05" size="1.016" layer="27" ratio="12"/>
+<element name="Q4" library="transistor" package="TO92" value="2N3904" x="59.69" y="24.765" smashed="yes">
+<attribute name="NAME" x="53.975" y="24.765" size="1.27" layer="25" ratio="12"/>
+<attribute name="VALUE" x="50.8" y="22.86" size="1.016" layer="27" ratio="12"/>
 </element>
 <element name="R23" library="rcl" package="0204/7" value="33k" x="72.39" y="52.07" smashed="yes" rot="R90">
@@
 <attribute name="VALUE" x="76.581" y="32.004" size="0.8128" layer="27" ratio="10"/>
 </element>
+<element name="R3" library="rcl" package="0204/7" value="1k" x="59.69" y="20.32" rot="R180"/>
 </elements>
 <signals>
@@
 <wire x1="72.39" y1="48.26" x2="72.39" y2="44.45" width="0.254" layer="1"/>
 <wire x1="72.39" y1="44.45" x2="71.12" y2="43.18" width="0.254" layer="16"/>
-<wire x1="71.12" y1="43.18" x2="71.12" y2="26.035" width="0.254" layer="16"/>
-<wire x1="71.12" y1="26.035" x2="66.04" y2="20.955" width="0.254" layer="16"/>
+<wire x1="71.12" y1="43.18" x2="71.12" y2="26.29098125" width="0.254" layer="16"/>
+<wire x1="71.12" y1="26.29098125" x2="67.05401875" y2="22.225" width="0.254" layer="16"/>
+<wire x1="67.05401875" y1="22.225" x2="64.77" y2="22.225" width="0.254" layer="16"/>
+<wire x1="64.77" y1="22.225" x2="62.23" y2="24.765" width="0.254" layer="16"/>
 </signal>
 <signal name="N$21">
 <contactref element="Q4" pad="2"/>
-<contactref element="IC7" pad="23"/>
-<wire x1="63.5" y1="20.955" x2="63.5" y2="16.51" width="0.254" layer="1"/>
+<contactref element="R3" pad="2"/>
+<wire x1="55.88" y1="20.32" x2="59.69" y2="24.13" width="0.254" layer="1"/>
+<wire x1="59.69" y1="24.13" x2="59.69" y2="24.765" width="0.254" layer="1"/>
 </signal>
 <signal name="N$5">
@@
 <contactref element="IC7" pad="24"/>
 </signal>
+<signal name="N$23">
+<contactref element="IC7" pad="23"/>
+<contactref element="R3" pad="1"/>
+<wire x1="63.5" y1="20.32" x2="63.5" y2="16.51" width="0.254" layer="1"/>
+</signal>
 </signals>
